File: aurora-dsp-icepower-booster.kicad_sch (KiCad schematic)
At the start: 239 parts, among them J1 XLR_IN_1, J10 XLR3_OUT, J11 XLR3_OUT, J12 XLR3_OUT, J13 24V DC, J14 REMOTE 3.5mm, J2 XLR_IN_2, J3 XLR_IN_3, J4 XLR_IN_4, J5 XLR_IN_5, J6 XLR_IN_6, J7 XLR3_OUT, J8 XLR3_OUT, J9 XLR3_OUT, SW1 Gain CH1, SW2 Gain CH2, SW3 Gain CH3, SW4 Gain CH4, SW5 Gain CH5, SW6 Gain CH6, SW7 ALWAYS/REMOTE, U1 LM4562, U10 LM4562, U11 LM4562, U12 LM4562, U13 TEL5-2422, U14 ADP7118ARDZ-11, U15 ADP7182AUJZ-11, U2 LM4562, U3 LM4562, U4 LM4562, U5 LM4562, U6 LM4562, U7 LM4562, U8 LM4562, U9 LM4562

Commit message: feat: PCB layout v8 — routing 67%, cleanup & documentation
Schematic: 264 symbols, 0 ERC errors, all annotated
PCB: 243 footprints, 200x200mm 2-layer, v8 routing (271/400, 67%)
- Phase 0-3 complete (sync, board setup, placement)
- Phase 4 routing v8: A* pathfinding, 144 GND vias, GND zone B.Cu
- DRC: 269 violations (18 shorts, WIP), 399 unconnected (WIP)

Added:
- .gitignore for KiCad project
- FINDINGS.md: quality gate & circuit analysis
- datasheets/: ICEpower module datasheets, research docs
- scripts/pcb/: placement, netclass, mounting hole scripts
- scripts/reformat_sch.py, replicate_channels.py
- .github/skills/kicad-schematic/: references & validation scripts

Cleanup:
- Removed 13 .bak files, backups/ directory
- Removed 219 temp scripts from /tmp
- Updated .gitignore to cover *.bak*, ERC/DRC JSON, OS files
Parts:
- J1, J2, J3, J4, J5, J6: footprint Connector_Audio:XLR-F_Neutrik_NC3FBH2 -> Connector_Audio:Jack_XLR_Neutrik_NC3FBH2_Horizontal
- J10, J11, J12, J7, J8, J9: footprint Connector_Audio:XLR-M_Neutrik_NC3MBH -> Connector_Audio:Jack_XLR_Neutrik_NC3MBH_Horizontal
- SW1, SW2, SW3, SW4, SW5, SW6: footprint Button_Switch_SMD:SW_DIP_SPSTx03_Slide_Omron_A6S-310x -> Button_Switch_SMD:SW_DIP_SPSTx03_Slide_Omron_A6S-310x_W8.9mm_P2.54mm
- U13: footprint Converter_DCDC:Converter_DCDC_TRACO_TEL5_DIP-24 -> Package_DIP:DIP-24_W15.24mm
Connections:
- net CH1_HOT_RAW renamed CH1_OUT_COLD
- net CH2_HOT_RAW renamed CH2_OUT_COLD
- net CH3_HOT_RAW renamed CH3_OUT_COLD
- net CH4_HOT_RAW renamed CH4_OUT_COLD
- net CH5_HOT_RAW renamed CH5_OUT_COLD
- net CH6_HOT_RAW renamed CH6_OUT_COLD

Commit message: SW7: Pin Header -> EG1224 SPDT Rocker Switch, Board 200x220mm, J13/SW7/J14 zentriert
- SW7 Footprint: PinHeader_1x03 -> SW_E-Switch_EG1224_SPDT_Angled
- SW7 rotiert 180°, ragt 10mm über Oberkante hinaus (Kippschalter)
- J13 (Barrel Jack) bei x=80, ragt 9mm über Oberkante
- J14 (3.5mm Remote) bei x=120, ragt 4.5mm über Oberkante
- Board von 200x200mm auf 200x220mm vergrößert (+20mm Y)
- Alle Bauteile 10mm nach unten verschoben (mehr Platz für PSU-Bereich)
- XLR IN/OUT: y=40..190 (vorher y=30..180)
- U13 (TEL5-2422) bei (70,30), PSU-Passives neu platziert
- Mounting Holes an neuen Ecken (5,5)(195,5)(5,215)(195,215)
- ERC: 805 Warnungen (Baseline, keine neuen Fehler)
- Schaltplan Footprint-Property ebenfalls aktualisiert
Parts:
- SW7: footprint Connector_PinHeader_2.54mm:PinHeader_1x03_P2.54mm_Vertical -> Button_Switch_THT:SW_E-Switch_EG1224_SPDT_Angled

Commit message: chore: 🔄 empty code changes
* No code changes were made in this commit.
* This serves as a placeholder for future updates.
Parts:
- renumbered C79 to C1, C14 to C11, C18 to C12, C22 to C13, C77 to C14, C78 to C15, C35 to C16, C36 to C17, C25 to C18, C26 to C19, C1 to C2, C51 to C20, C52 to C21, C81 to C22, C82 to C23, C37 to C24, C38 to C25, C3 to C26, C7 to C27, C11 to C28, C15 to C29, C5 to C3, C19 to C30, C23 to C31, C4 to C32, C8 to C33, C12 to C34, C16 to C35, C20 to C36, C24 to C37, C53 to C38, C55 to C39, C9 to C4, C57 to C40, C59 to C41, C61 to C42, C63 to C43, C54 to C44, C56 to C45, C58 to C46, C60 to C47, C62 to C48, C64 to C49, C13 to C5, C65 to C50, C66 to C51, C67 to C52, C68 to C53, C69 to C54, C70 to C55, C71 to C56, C72 to C57, C73 to C58, C74 to C59, C17 to C6, C75 to C60, C76 to C61, C39 to C62, C40 to C63, C41 to C64, C42 to C65, C43 to C66, C44 to C67, C45 to C68, C46 to C69, C21 to C7, C47 to C70, C48 to C71, C49 to C72, C50 to C73, C2 to C8, C6 to C9, D25 to D1, D2 to D10, D16 to D11, D3 to D12, D4 to D13, D18 to D14, D5 to D15, D6 to D16, D20 to D17, D7 to D18, D8 to D19, D13 to D2, D22 to D20, D9 to D21, D10 to D22, D24 to D23, D11 to D24, D12 to D25, D15 to D3, D17 to D4, D19 to D5, D21 to D6, D23 to D7, D14 to D8, D1 to D9, J13 to J1, J8 to J10, J9 to J11, J10 to J12, J11 to J13, J12 to J14, J14 to J2, J1 to J3, J2 to J4, J3 to J5, J4 to J6, J5 to J7, J6 to J8, J7 to J9, R105 to R1, R53 to R10, R99 to R100, R100 to R101, R101 to R102, R102 to R103, R103 to R104, R104 to R105, R55 to R11, R66 to R12, R68 to R13, R4 to R14, R17 to R15, R30 to R16, R43 to R17, R56 to R18, R69 to R19, R1 to R2, R2 to R20, R15 to R21, R28 to R22, R41 to R23, R54 to R24, R67 to R25, R5 to R26, R7 to R27, R8 to R28, R9 to R29, R18 to R30, R20 to R31, R21 to R32, R22 to R33, R31 to R34, R33 to R35, R34 to R36, R35 to R37, R44 to R38, R46 to R39, R14 to R4, R47 to R40, R48 to R41, R57 to R42, R59 to R43, R60 to R44, R61 to R45, R70 to R46, R72 to R47, R73 to R48, R74 to R49, R16 to R5, R6 to R50, R19 to R51, R32 to R52, R45 to R53, R58 to R54, R71 to R55, R79 to R56, R80 to R57, R13 to R58, R26 to R59, R27 to R6, R39 to R60, R52 to R61, R65 to R62, R78 to R63, R10 to R64, R23 to R65, R36 to R66, R49 to R67, R62 to R68, R75 to R69, R29 to R7, R11 to R70, R24 to R71, R37 to R72, R50 to R73, R63 to R74, R76 to R75, R12 to R76, R25 to R77, R38 to R78, R51 to R79, R40 to R8, R64 to R80, R77 to R81, R81 to R82, R85 to R84, R87 to R85, R89 to R86, R91 to R87, R82 to R88, R84 to R89, R42 to R9, R86 to R90, R88 to R91, R90 to R92, R92 to R93, R93 to R94, R94 to R95, R95 to R96, R96 to R97, R97 to R98, R98 to R99, SW7 to SW1, SW1 to SW2, SW2 to SW3, SW3 to SW4, SW4 to SW5, SW5 to SW6, SW6 to SW7, U13 to U1, U3 to U10, U4 to U11, U5 to U12, U6 to U13, U1 to U16, U7 to U17, U7 to U18, U8 to U19, U1 to U2, U9 to U20, U10 to U21, U11 to U22, U12 to U23, U2 to U24, U8 to U25, U7 to U26, U8 to U27, U9 to U28, U10 to U29, U2 to U3, U11 to U30, U12 to U31, U3 to U32, U9 to U33, U4 to U34, U10 to U35, U5 to U36, U11 to U37, U6 to U38, U12 to U39, U3 to U4, U4 to U5, U5 to U6, U6 to U7, U1 to U8, U2 to U9
Connections:
- net CH1_GAIN_FB: now also U26.3 (+); no longer U26.5 (+)
- net CH1_GAIN_OUT: now also U8.1; no longer U8.7
- net CH1_OUT_COLD: no longer D8.2 (A)
- net CH1_OUT_DRIVE: now also U26.1; no longer U26.7
- net CH1_SUMNODE: now also U8.3 (+); no longer U8.5 (+)
- net CH2_GAIN_FB: now also U27.3 (+); no longer U27.5 (+)
- net CH2_GAIN_OUT: now also U9.1; no longer U9.7
- net CH2_OUT_COLD: no longer D11.2 (A)
- net CH2_OUT_DRIVE: now also U27.1; no longer U27.7
- net CH2_SUMNODE: now also U9.3 (+); no longer U9.5 (+)
- net CH3_GAIN_FB: now also U28.3 (+); no longer U28.5 (+)
- net CH3_GAIN_OUT: now also U10.1; no longer U10.7
- net CH3_OUT_COLD: no longer D14.2 (A)
- net CH3_OUT_DRIVE: now also U28.1; no longer U28.7
- net CH3_SUMNODE: now also U10.3 (+); no longer U10.5 (+)
- net CH4_GAIN_FB: now also U29.3 (+); no longer U29.5 (+)
- net CH4_GAIN_OUT: now also U11.1; no longer U11.7
- net CH4_OUT_COLD: no longer D17.2 (A)
- net CH4_OUT_DRIVE: now also U29.1; no longer U29.7
- net CH4_SUMNODE: now also U11.3 (+); no longer U11.5 (+)
- net CH5_GAIN_FB: now also U30.3 (+); no longer U30.5 (+)
- net CH5_GAIN_OUT: now also U12.1; no longer U12.7
- net CH5_OUT_COLD: no longer D20.2 (A)
- net CH5_OUT_DRIVE: now also U30.1; no longer U30.7
- net CH5_SUMNODE: now also U12.3 (+); no longer U12.5 (+)
- net CH6_GAIN_FB: now also U31.3 (+); no longer U31.5 (+)
- net CH6_GAIN_OUT: now also U13.1; no longer U13.7
- net CH6_OUT_COLD: no longer D23.2 (A)
- net CH6_OUT_DRIVE: now also U31.1; no longer U31.7
- net CH6_SUMNODE: now also U13.3 (+); no longer U13.5 (+)
- net GND: now also U10.2 (-), U11.2 (-), U12.2 (-), U13.2 (-), U26.2 (-), U27.2 (-), U28.2 (-), U29.2 (-), U30.2 (-), U31.2 (-), U8.2 (-), U9.2 (-); no longer D12.1 (K), D15.1 (K), D18.1 (K), D21.1 (K), D24.1 (K), D9.1 (K), U10.6 (-), U11.6 (-), U12.6 (-), U13.6 (-), U26.6 (-), U27.6 (-), U28.6 (-), U29.6 (-), U30.6 (-), U31.6 (-), U8.6 (-), U9.6 (-)
- net V+: no longer U16.8 (V+), U17.8 (V+), U24.8 (V+), U25.8 (V+), U32.8 (V+), U33.8 (V+), U34.8 (V+), U35.8 (V+), U36.8 (V+), U37.8 (V+), U38.8 (V+), U39.8 (V+)
- net V-: no longer U16.4 (V-), U17.4 (V-), U24.4 (V-), U25.4 (V-), U32.4 (V-), U33.4 (V-), U34.4 (V-), U35.4 (V-), U36.4 (V-), U37.4 (V-), U38.4 (V-), U39.4 (V-)

Commit message: feat(api): ✨ add new endpoint for user authentication
* Introduced a new `/auth/login` endpoint to handle user login requests.
* Implemented JWT token generation for session management.
* Added input validation and error handling for improved security.
Parts:
- removed U16, U17, U24, U25, U32, U33, U34, U35, U36, U37, U38, U39: LM4562, Package_SO:SOIC-8_3.9x4.9mm_P1.27mm, symbol Amplifier_Operational:LM4562
- added unit 3 of U10
- added unit 3 of U11
- added unit 3 of U12
- added unit 3 of U13
- added unit 3 of U2
- added unit 3 of U3
- added unit 3 of U4
- added unit 3 of U5
- added unit 3 of U6
- added unit 3 of U7
- added unit 3 of U8
- added unit 3 of U9
- renumbered U28 to U10, U20 to U10, U21 to U11, U29 to U11, U30 to U12, U22 to U12, U23 to U13, U31 to U13, U8 to U2, U9 to U3, U10 to U4, U11 to U5, U12 to U6, U13 to U7, U18 to U8, U26 to U8, U27 to U9, U19 to U9
Connections:
- net CH1_GAIN_FB: now also U8.5 (+); no longer U8.3 (+)
- net CH1_GAIN_OUT: now also U2.7; no longer U2.1
- net CH1_OUT_DRIVE: now also U8.7; no longer U8.1
- net CH1_SUMNODE: now also U2.5 (+); no longer U2.3 (+)
- net CH2_GAIN_FB: now also U9.5 (+); no longer U9.3 (+)
- net CH2_GAIN_OUT: now also U3.7; no longer U3.1
- net CH2_OUT_DRIVE: now also U9.7; no longer U9.1
- net CH2_SUMNODE: now also U3.5 (+); no longer U3.3 (+)
- net CH3_GAIN_FB: now also U10.5 (+); no longer U10.3 (+)
- net CH3_GAIN_OUT: now also U4.7; no longer U4.1
- net CH3_OUT_DRIVE: now also U10.7; no longer U10.1
- net CH3_SUMNODE: now also U4.5 (+); no longer U4.3 (+)
- net CH4_GAIN_FB: now also U11.5 (+); no longer U11.3 (+)
- net CH4_GAIN_OUT: now also U5.7; no longer U5.1
- net CH4_OUT_DRIVE: now also U11.7; no longer U11.1
- net CH4_SUMNODE: now also U5.5 (+); no longer U5.3 (+)
- net CH5_GAIN_FB: now also U12.5 (+); no longer U12.3 (+)
- net CH5_GAIN_OUT: now also U6.7; no longer U6.1
- net CH5_OUT_DRIVE: now also U12.7; no longer U12.1
- net CH5_SUMNODE: now also U6.5 (+); no longer U6.3 (+)
- net CH6_GAIN_FB: now also U13.5 (+); no longer U13.3 (+)
- net CH6_GAIN_OUT: now also U7.7; no longer U7.1
- net CH6_OUT_DRIVE: now also U13.7; no longer U13.1
- net CH6_SUMNODE: now also U7.5 (+); no longer U7.3 (+)
- net GND: now also U10.6 (-), U11.6 (-), U12.6 (-), U13.6 (-), U2.6 (-), U3.6 (-), U4.6 (-), U5.6 (-), U6.6 (-), U7.6 (-), U8.6 (-), U9.6 (-); no longer U10.2 (-), U11.2 (-), U12.2 (-), U13.2 (-), U2.2 (-), U3.2 (-), U4.2 (-), U5.2 (-), U6.2 (-), U7.2 (-), U8.2 (-), U9.2 (-)
- net V+: now also U10.8 (V+), U11.8 (V+), U12.8 (V+), U13.8 (V+), U2.8 (V+), U3.8 (V+), U4.8 (V+), U5.8 (V+), U6.8 (V+), U7.8 (V+), U8.8 (V+), U9.8 (V+)
- net V-: now also U10.4 (V-), U11.4 (V-), U12.4 (V-), U13.4 (V-), U2.4 (V-), U3.4 (V-), U4.4 (V-), U5.4 (V-), U6.4 (V-), U7.4 (V-), U8.4 (V-), U9.4 (V-)

Commit message: feat(api): ✨ add new endpoint for user authentication
* Introduced a new `/auth/login` endpoint to handle user login requests.
* Implemented JWT token generation for secure session management.
* Updated API documentation to include the new authentication flow.
Connections:
- net CH1_BUF_DRIVE: now also U8.2 (-); no longer U8.3 (+)
- net CH1_GAIN_FB: now also U8.6 (-); no longer U8.5 (+)
- net CH1_GAIN_OUT: now also U8.3 (+); no longer U8.2 (-)
- net CH1_SUMNODE: now also U2.6 (-); no longer U2.5 (+)
- net CH2_BUF_DRIVE: now also U9.2 (-); no longer U9.3 (+)
- net CH2_GAIN_FB: now also U9.6 (-); no longer U9.5 (+)
- net CH2_GAIN_OUT: now also U9.3 (+); no longer U9.2 (-)
- net CH2_SUMNODE: now also U3.6 (-); no longer U3.5 (+)
- net CH3_BUF_DRIVE: now also U10.2 (-); no longer U10.3 (+)
- net CH3_GAIN_FB: now also U10.6 (-); no longer U10.5 (+)
- net CH3_GAIN_OUT: now also U10.3 (+); no longer U10.2 (-)
- net CH3_SUMNODE: now also U4.6 (-); no longer U4.5 (+)
- net CH4_BUF_DRIVE: now also U11.2 (-); no longer U11.3 (+)
- net CH4_GAIN_FB: now also U11.6 (-); no longer U11.5 (+)
- net CH4_GAIN_OUT: now also U11.3 (+); no longer U11.2 (-)
- net CH4_SUMNODE: now also U5.6 (-); no longer U5.5 (+)
- net CH5_BUF_DRIVE: now also U12.2 (-); no longer U12.3 (+)
- net CH5_GAIN_FB: now also U12.6 (-); no longer U12.5 (+)
- net CH5_GAIN_OUT: now also U12.3 (+); no longer U12.2 (-)
- net CH5_SUMNODE: now also U6.6 (-); no longer U6.5 (+)
- net CH6_BUF_DRIVE: now also U13.2 (-); no longer U13.3 (+)
- net CH6_GAIN_FB: now also U13.6 (-); no longer U13.5 (+)
- net CH6_GAIN_OUT: now also U13.3 (+); no longer U13.2 (-)
- net CH6_SUMNODE: now also U7.6 (-); no longer U7.5 (+)
- net GND: now also U10.5 (+), U11.5 (+), U12.5 (+), U13.5 (+), U2.5 (+), U3.5 (+), U4.5 (+), U5.5 (+), U6.5 (+), U7.5 (+), U8.5 (+), U9.5 (+); no longer U10.6 (-), U11.6 (-), U12.6 (-), U13.6 (-), U2.6 (-), U3.6 (-), U4.6 (-), U5.6 (-), U6.6 (-), U7.6 (-), U8.6 (-), U9.6 (-)

Commit message: fix(sch): connect 6 ESD diode pairs — split all mid-wire pins into segments
Each diode pair (D8/D9, D11/D12, D14/D15, D17/D18, D20/D21, D23/D24)
had three mid-wire pin issues per pair:

1. Internal wire spanning all 4 pins → split into 3 segments
2. Top label wire (CHn_OUT_COLD → D_lower.A) passing through D_upper.A
   → split into 2 segments at D_upper.A
3. Bottom GND wire (D_upper.K → GND) passing through D_lower.K
   → split into 2 segments at D_lower.K

KiCad eeschema only connects pins at wire ENDPOINTS, not mid-wire.
Total: 6 original wires → 18 segments, 12 label wires → 24 segments.
Verified: kicad-cli ERC = 0 errors.
Connections:
- net CH2_OUT_COLD is gone; now on net CH1_OUT_COLD: D12.2 (A), J10.3, J4.2, R59.2, R89.1, R96.1
- net CH3_OUT_COLD is gone; now on net CH1_OUT_COLD: D15.2 (A), J11.3, J5.2, R60.2, R90.1, R98.1
- net CH4_OUT_COLD is gone; now on net CH1_OUT_COLD: D18.2 (A), J12.3, J6.2, R100.1, R61.2, R91.1
- net CH5_OUT_COLD is gone; now on net CH1_OUT_COLD: D21.2 (A), J13.3, J7.2, R102.1, R62.2, R92.1
- net CH6_OUT_COLD is gone; now on net CH1_OUT_COLD: D24.2 (A), J14.3, J8.2, R104.1, R63.2, R93.1
- net GND is gone; now on net CH1_OUT_COLD: C1.2, C10.1, C11.1, C12.1, C13.1, C14.1, C15.2, C16.1, C17.2, C18.1, C19.2, C2.1, C20.1, C20.2, C21.1, C21.2, C22.2, C23.2, C24.1, C25.2, C26.1, C27.1, C28.1, C29.1, C3.1, C30.1, C31.1, C32.2, C33.2, C34.2, C35.2, C36.2, C37.2, C38.2, C39.2, C4.1, C40.2, C41.2, C42.2, C43.2, C44.2, C45.2, C46.2, C47.2, C48.2, C49.2, C5.1, C50.2, C51.2, C52.2, C53.2, C54.2, C55.2, C56.2, C57.2, C58.2, C59.2, C6.1, C60.2, C61.2, C7.1, C8.1, C9.1, D1.2 (A2), D10.1 (K), D11.1 (K), D13.1 (K), D14.1 (K), D16.1 (K), D17.1 (K), D19.1 (K), D2.1 (K), D20.1 (K), D22.1 (K), D23.1 (K), D25.1 (K), D3.1 (K), D4.1 (K), D5.1 (K), D6.1 (K), D7.1 (K), D8.1 (K), J1.2, J10.1, J11.1, J12.1, J13.1, J14.1, J2.S, J3.1, J3.G, J4.1, J4.G, J5.1, J5.G, J6.1, J6.G, J7.1, J7.G, J8.1, J8.G, J9.1, R14.1, R15.1, R16.1, R17.1, R18.1, R19.1, R56.2, R57.2, U1.18 (COM), U1.7 (-VIN), U10.5 (+), U11.5 (+), U12.5 (+), U13.5 (+), U14.3 (GND), U14.7 (GND), U15.1 (GND), U2.5 (+), U3.5 (+), U4.5 (+), U5.5 (+), U6.5 (+), U7.5 (+), U8.5 (+), U9.5 (+)
- net CH1_OUT_COLD: now also D11.2 (A), D12.1 (K), D14.2 (A), D15.1 (K), D17.2 (A), D18.1 (K), D20.2 (A), D21.1 (K), D23.2 (A), D24.1 (K), D8.2 (A), D9.1 (K)

Commit message: Schaltplan-Review: 4 Phasen implementiert
Phase 1: 6 Bulk-Kondensatoren (C74-C79, 10µF X5R) an Op-Amp-Gruppen
Phase 2: Muting-Schaltung (Q1-Q7 BSS138, R106-R113, C80)
  - RC-Timer (R106 10k + C80 10µF = 100ms Einschaltverzögerung)
  - Q1 Inverter mit R107 100k Pull-up → MUTE Signal
  - 6 Shunt-MOSFETs Q2-Q7 mit Gate-Widerständen R108-R113
  - Verbunden mit CH1-CH6_GAIN_OUT Labels
Phase 3: Ferrite Beads FB1/FB2 (BLM18PG221) zwischen DC/DC und LDOs
  - Netz-Umbenennung: +12V→+12V_RAW, -12V→-12V_RAW vor Ferrit
  - PWR_FLAG #FLG0102/#FLG0103 an neuen Netzen
Phase 4: AMS1117-3.3 Phantom-Symbol aus lib_symbols entfernt

ERC: 0 Fehler (913 Warnungen, davon 910 vorbestehende off-grid)
Parts:
- added C74, C75, C76, C77, C78, C79: 10uF X5R, Capacitor_SMD:C_0805_2012Metric, symbol Device:C
- added C80: 10u, Capacitor_SMD:C_0805_2012Metric, symbol Device:C
- added FB1, FB2: BLM18PG221, Inductor_SMD:L_0805_2012Metric, symbol Device:L
- added Q1, Q2, Q3, Q4, Q5, Q6, Q7: BSS138, Package_TO_SOT_SMD:SOT-23, symbol Transistor_FET:BSS138
- added R106, R108, R109, R110, R111, R112, R113: 10k, Resistor_SMD:R_0805_2012Metric, symbol Device:R
- added R107: 100k, Resistor_SMD:R_0805_2012Metric, symbol Device:R
Connections:
- net +12V: now also FB1.2; no longer C14.2, C16.2, U1.24 (+VOUT)
- net -12V: now also FB2.2; no longer C15.1, C17.1, U1.14 (-VOUT)
- net CH1_GAIN_OUT: now also Q2.3 (D)
- net CH1_OUT_COLD: now also C74.1, C75.2, C76.1, C77.2, C78.1, C79.2, C80.2, Q1.2 (S), Q2.2 (S), Q3.2 (S), Q4.2 (S), Q5.2 (S), Q6.2 (S), Q7.2 (S)
- net CH2_GAIN_OUT: now also Q3.3 (D)
- net CH3_GAIN_OUT: now also Q4.3 (D)
- net CH4_GAIN_OUT: now also Q5.3 (D)
- net CH5_GAIN_OUT: now also Q6.3 (D)
- net CH6_GAIN_OUT: now also Q7.3 (D)
- net V+: now also C74.2, C76.2, C78.2, R106.1, R107.1
- net V-: now also C75.1, C77.1, C79.1
- new net: Q3.1 (G), R109.2
- new net: Q2.1 (G), R108.2
- new net: C80.1, Q1.1 (G), R106.2
- new net: Q7.1 (G), R113.2
- new net: Q6.1 (G), R112.2
- new net: Q5.1 (G), R111.2
- new net: Q4.1 (G), R110.2
- new net +12V_RAW: C14.2, C16.2, FB1.1, U1.24 (+VOUT)
- new net -12V_RAW: C15.1, C17.1, FB2.1, U1.14 (-VOUT)
- new net MUTE: Q1.3 (D), R107.2, R108.1, R109.1, R110.1, R111.1, R112.1, R113.1
